Commit message: modified joint constraints for better IK

File: resources/pepper/pepper.urdf (robot description, URDF)
Before this commit: robot JulietteY20MP, 84 links, 83 joints
Joints:
- joint RElbowYaw: limit lower=-2.08567 upper=2.08567 effort=5.428 velocity=7.33998 -> lower=0.5854 upper=0.9854 effort=5.428 velocity=7.33998
- joint RShoulderRoll: limit lower=-1.56207 upper=-0.00872665 effort=2.666 velocity=9.22756 -> lower=-1.56207 upper=-0.109 effort=2.666 velocity=9.22756

Commit message: made setting changes

File: resources/pepper/pepper.urdf (robot description, URDF)
Before this commit: robot JulietteY20MP, 84 links, 83 joints
Joints:
- joint RElbowYaw: limit lower=0.5854 upper=0.9854 effort=5.428 velocity=7.33998 -> lower=-2.08567 upper=2.08567 effort=5.428 velocity=7.33998
- joint RShoulderRoll: limit lower=-1.56207 upper=-0.109 effort=2.666 velocity=9.22756 -> lower=-1.56207 upper=-0.00872665 effort=2.666 velocity=9.22756
